File: Electronics/HC-base_revA.sch (EAGLE design)
At the start: 35 parts, among them T2 BSS138, T3 BSS138, T4 BSS138, T5 BSS138, U2 NRF24L01, U3 OLED128X64

Commit message: modified: diagram and pcb
Parts:
- removed C3: (no value), rcl:CPOL-EU153CLV-1012
- removed R1: 0R\, 1_domaci:R'2'
- added U$1, U$2, U$3: CORNER, 1_domaci:CORNER
- C4: device 1_domaci:C-POLY'10MM' -> 1_domaci:C-POLY'6.5MM'
Connections:
- new net N$21: U1.GND@39, U2.GND
- net BUT1: now also U1.GPIO17; no longer U1.GPIO14
- net GND: no longer R1.P$1, R1.P$2, U1.GND@34, U2.GND
- net LED3: now also U1.GPIO22; no longer U1.GPIO18
- net LED4: now also U1.GPIO27; no longer U1.GPIO15
Other:
- moved on the sheet: BUT1, BUT2, LED1, LED2, LED3, LED4, R10, R11, R12, R13, R14, R15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

Commit message: modified: finished PCB
Parts:
- R12: value 680R -> 560R
- R4, R6: value 680R -> 3k3
- R9: value 680R -> 1k
Changed lines of the file:
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@@
 <grid distance="0.1" unitdist="inch" unit="inch" style="lines" multiple="1" display="no" altdistance="0.01" altunitdist="inch" altunit="inch"/>
 <layers>
-<layer number="1" name="Top" color="4" fill="1" visible="yes" active="no"/>
-<layer number="16" name="Bottom" color="1" fill="1" visible="yes" active="no"/>
-<layer number="17" name="Pads" color="2" fill="1" visible="yes" active="no"/>
-<layer number="18" name="Vias" color="2" fill="1" visible="yes" active="no"/>
-<layer number="19" name="Unrouted" color="6" fill="1" visible="yes" active="no"/>
-<layer number="20" name="Dimension" color="15" fill="1" visible="yes" active="no"/>
-<layer number="21" name="tPlace" color="7" fill="1" visible="yes" active="no"/>
-<layer number="22" name="bPlace" color="7" fill="1" visible="yes" active="no"/>
-<layer number="23" name="tOrigins" color="15" fill="1" visible="yes" active="no"/>
-<layer number="24" name="bOrigins" color="15" fill="1" visible="yes" active="no"/>
-<layer number="25" name="tNames" color="7" fill="1" visible="yes" active="no"/>
-<layer number="26" name="bNames" color="7" fill="1" visible="yes" active="no"/>
-<layer number="27" name="tValues" color="7" fill="1" visible="yes" active="no"/>
-<layer number="28" name="bValues" color="7" fill="1" visible="yes" active="no"/>
+<layer number="1" name="Top" color="4" fill="1" visible="no" active="no"/>
+<layer number="16" name="Bottom" color="1" fill="1" visible="no" active="no"/>
+<layer number="17" name="Pads" color="2" fill="1" visible="no" active="no"/>
+<layer number="18" name="Vias" color="2" fill="1" visible="no" active="no"/>
+<layer number="19" name="Unrouted" color="6" fill="1" visible="no" active="no"/>
+<layer number="20" name="Dimension" color="15" fill="1" visible="no" active="no"/>
+<layer number="21" name="tPlace" color="7" fill="1" visible="no" active="no"/>
+<layer number="22" name="bPlace" color="7" fill="1" visible="no" active="no"/>
+<layer number="23" name="tOrigins" color="15" fill="1" visible="no" active="no"/>
+<layer number="24" name="bOrigins" color="15" fill="1" visible="no" active="no"/>
+<layer number="25" name="tNames" color="7" fill="1" visible="no" active="no"/>
+<layer number="26" name="bNames" color="7" fill="1" visible="no" active="no"/>
+<layer number="27" name="tValues" color="7" fill="1" visible="no" active="no"/>
+<layer number="28" name="bValues" color="7" fill="1" visible="no" active="no"/>
 <layer number="29" name="tStop" color="7" fill="3" visible="no" active="no"/>
 <layer number="30" name="bStop" color="7" fill="6" visible="no" active="no"/>
@@
 <layer number="35" name="tGlue" color="7" fill="4" visible="no" active="no"/>
 <layer number="36" name="bGlue" color="7" fill="5" visible="no" active="no"/>
-<layer number="37" name="tTest" color="7" fill="1" visible="yes" active="no"/>
-<layer number="38" name="bTest" color="7" fill="1" visible="yes" active="no"/>
+<layer number="37" name="tTest" color="7" fill="1" visible="no" active="no"/>
+<layer number="38" name="bTest" color="7" fill="1" visible="no" active="no"/>
 <layer number="39" name="tKeepout" color="4" fill="11" visible="no" active="no"/>
 <layer number="40" name="bKeepout" color="1" fill="11" visible="no" active="no"/>
@@
 <layer number="44" name="Drills" color="7" fill="1" visible="no" active="no"/>
 <layer number="45" name="Holes" color="7" fill="1" visible="no" active="no"/>
-<layer number="46" name="Milling" color="3" fill="1" visible="yes" active="no"/>
-<layer number="47" name="Measures" color="7" fill="1" visible="yes" active="no"/>
-<layer number="48" name="Document" color="7" fill="1" visible="yes" active="no"/>
-<layer number="49" name="Reference" color="7" fill="1" visible="yes" active="no"/>
-<layer number="50" name="dxf" color="7" fill="1" visible="yes" active="no"/>
-<layer number="51" name="tDocu" color="7" fill="1" visible="yes" active="no"/>
-<layer number="52" name="bDocu" color="7" fill="1" visible="yes" active="no"/>
-<layer number="53" name="tGND_GNDA" color="7" fill="9" visible="yes" active="no"/>
-<layer number="54" name="bGND_GNDA" color="1" fill="9" visible="yes" active="no"/>
-<layer number="56" name="wert" color="7" fill="1" visible="yes" active="no"/>
-<layer number="57" name="tCAD" color="7" fill="1" visible="yes" active="no"/>
+<layer number="46" name="Milling" color="3" fill="1" visible="no" active="no"/>
+<layer number="47" name="Measures" color="7" fill="1" visible="no" active="no"/>
+<layer number="48" name="Document" color="7" fill="1" visible="no" active="no"/>
+<layer number="49" name="Reference" color="7" fill="1" visible="no" active="no"/>
+<layer number="50" name="dxf" color="7" fill="1" visible="no" active="no"/>
+<layer number="51" name="tDocu" color="7" fill="1" visible="no" active="no"/>
+<layer number="52" name="bDocu" color="7" fill="1" visible="no" active="no"/>
+<layer number="53" name="tGND_GNDA" color="7" fill="9" visible="no" active="no"/>
+<layer number="54" name="bGND_GNDA" color="1" fill="9" visible="no" active="no"/>
+<layer number="56" name="wert" color="7" fill="1" visible="no" active="no"/>
+<layer number="57" name="tCAD" color="7" fill="1" visible="no" active="no"/>
 <layer number="90" name="Modules" color="5" fill="1" visible="yes" active="yes"/>
 <layer number="91" name="Nets" color="2" fill="1" visible="yes" active="yes"/>
@@
 <part name="T2" library="1_domaci" deviceset="BSS138" device="" value="BSS138"/>
 <part name="LED1" library="1_domaci" deviceset="LED" device="'SMD'" value="GREEN"/>
-<part name="R4" library="1_domaci" deviceset="R" device="'2'" value="680R"/>
+<part name="R4" library="1_domaci" deviceset="R" device="'2'" value="3k3"/>
 <part name="+3V4" library="1_domaci" deviceset="+3V3" device=""/>
 <part name="GND5" library="1_domaci" deviceset="GND" device=""/>
@@
 <part name="T3" library="1_domaci" deviceset="BSS138" device="" value="BSS138"/>
 <part name="LED2" library="1_domaci" deviceset="LED" device="'SMD'" value="GREEN"/>
-<part name="R6" library="1_domaci" deviceset="R" device="'2'" value="680R"/>
+<part name="R6" library="1_domaci" deviceset="R" device="'2'" value="3k3"/>
 <part name="+3V5" library="1_domaci" deviceset="+3V3" device=""/>
 <part name="GND6" library="1_domaci" deviceset="GND" device=""/>
@@
 <part name="T4" library="1_domaci" deviceset="BSS138" device="" value="BSS138"/>
 <part name="LED3" library="1_domaci" deviceset="LED" device="'SMD'" value="ORANGE"/>
-<part name="R9" library="1_domaci" deviceset="R" device="'2'" value="680R"/>
+<part name="R9" library="1_domaci" deviceset="R" device="'2'" value="1k"/>
 <part name="+3V6" library="1_domaci" deviceset="+3V3" device=""/>
 <part name="GND7" library="1_domaci" deviceset="GND" device=""/>
@@
 <part name="T5" library="1_domaci" deviceset="BSS138" device="" value="BSS138"/>
 <part name="LED4" library="1_domaci" deviceset="LED" device="'SMD'" value="RED"/>
-<part name="R12" library="1_domaci" deviceset="R" device="'2'" value="680R"/>
+<part name="R12" library="1_domaci" deviceset="R" device="'2'" value="560R"/>
 <part name="+3V7" library="1_domaci" deviceset="+3V3" device=""/>
 <part name="GND8" library="1_domaci" deviceset="GND" device=""/>
